Commit message: [#333] Replacing lgsvl_odom with gnss/gnss_odom and lidar_back with lidar_rear.

File: src/urdf/lexus_rx_450h_description/urdf/lexus_rx_450h.urdf (robot description, URDF)
Before this commit: robot lexus_rx_450h, 3 links, 2 joints
Links:
- removed link lidar_back
- added link lidar_rear, mass 0.1; collision cylinder length=0.0869 radius=0.05165; visual cylinder length=0.0869 radius=0.05165
Joints:
- removed joint lidar_back_joint
- added joint lidar_rear_joint: type fixed, parent base_link, child lidar_rear, origin xyz=0.308 -0.022 1.49 rpy=0 0 0

Commit message: [#339] Adding CoG link to URDF as nav_base.

File: src/urdf/lexus_rx_450h_description/urdf/lexus_rx_450h.urdf (robot description, URDF)
Before this commit: robot lexus_rx_450h, 3 links, 2 joints
Links:
- added link nav_base
Joints:
- added joint nav_base_joint: type fixed, parent base_link, child nav_base, origin xyz=1.5618 0 0 rpy=0 0 0

Commit message: [#1289] Add the camera to the urdf file

File: src/urdf/lexus_rx_450h_description/urdf/lexus_rx_450h.urdf (robot description, URDF)
Before this commit: robot lexus_rx_450h, 6 links, 5 joints
Links:
- added link camera, mass 0.1; collision box size=0.05 0.1 0.1; visual box size=0.05 0.1 0.1
Joints:
- added joint camera_joint: type fixed, parent base_link, child camera, origin xyz=-0.2 0 1.7 rpy=0 0 0

Commit message: Add orientation to camera

File: src/urdf/lexus_rx_450h_description/urdf/lexus_rx_450h.urdf (robot description, URDF)
Before this commit: robot lexus_rx_450h, 7 links, 6 joints
Joints:
- joint camera_joint: origin xyz=-0.2 0 1.7 rpy=0 0 0 -> xyz=-0.2 0 1.7 rpy=1.571 1.571 0

Commit message: [#1338] Add support for multiple cameras in the object tracker

File: src/urdf/lexus_rx_450h_description/urdf/lexus_rx_450h.urdf (robot description, URDF)
Before this commit: robot lexus_rx_450h, 7 links, 6 joints
Links:
- removed link camera
- added link camera_left, mass 0.1; collision box size=0.05 0.1 0.1; visual box size=0.05 0.1 0.1
- added link camera_right, mass 0.1; collision box size=0.05 0.1 0.1; visual box size=0.05 0.1 0.1
Joints:
- removed joint camera_joint
- added joint camera_left_joint: type fixed, parent base_link, child camera_left, origin xyz=1.75 -0.5 1.25 rpy=-1.571 0 -0.78539
- added joint camera_right_joint: type fixed, parent base_link, child camera_right, origin xyz=1.75 0.5 1.25 rpy=-1.571 0 -2.356194
