Commit message: [#1338] Change projection params & add params for single camera

File: src/urdf/lexus_rx_450h_description/urdf/lexus_rx_450h_dual_camera.urdf (robot description, URDF)
Before this commit: robot lexus_rx_450h, 7 links, 6 joints
Links:
- removed link camera
- added link camera_left, mass 0.1; collision box size=0.05 0.1 0.1; visual box size=0.05 0.1 0.1
- added link camera_right, mass 0.1; collision box size=0.05 0.1 0.1; visual box size=0.05 0.1 0.1
Joints:
- removed joint camera_joint
- added joint camera_left_joint: type fixed, parent base_link, child camera_left, origin xyz=1.75 0.5 1.25 rpy=-1.571 0 -0.78539
- added joint camera_right_joint: type fixed, parent base_link, child camera_right, origin xyz=1.75 -0.5 1.25 rpy=-1.571 0 -2.356194
